File: RE3RT4Prog.kicad_pcb (KiCad board)
At the start: 2 copper layers, 130 x 100 mm, 69 parts, among them J1 Conn_01x08, J2 Conn_01x08, J3 DE9_Receptacle_MountingHoles, J4 +5V, J5 GND, J6 PicKit, J7 Barrel_Jack_MountingPin, Q1 BD140, Q2 2N7000, Q3 2N7000, Q4 2N7000, U1 DG408, U2 155RE3, U3 556RT4, U4 74HC164, U6 PIC18F26K22-xSP, U7 MAX232, Y1 7.3728

Commit message: Work in progress, close
Parts:
- removed R1, R4: R, Resistor_THT:R_Axial_DIN0207_L6.3mm_D2.5mm_P10.16mm_Horizontal
- moved R12 15.0 mm to (97.8, 104.3)
- moved Q4 5.89 mm to (102.5, 96.3)
- moved R13 5.39 mm to (108.4, 89.3)
- moved J1 3.19 mm to (82.0, 31.0)
- moved U1 1.38 mm to (107.7, 33.5)
- moved J2 0.32 mm to (57.3, 48.8)
Routing:
- net /SER: track 0.00 -> 160.1 mm, vias 0 -> 2
- net /CE: track 0.00 -> 132.6 mm, vias 0 -> 1
- net /B0: track 14.3 -> 123.0 mm, vias 0 -> 1
- net /A0: track 0.00 -> 96.6 mm, vias 0 -> 5
- net /RD: track 38.1 -> 129.3 mm, vias 0 -> 1
- net /D4: track 0.00 -> 88.7 mm, vias 0 -> 3
- net /CLK: track 33.2 -> 120.1 mm, vias 0 -> 4
- net /B1: track 8.38 -> 90.6 mm, vias 0 -> 2
- net /D1: track 0.00 -> 76.7 mm, vias 0 -> 2
- net /B2: track 9.40 -> 85.8 mm, vias 0 -> 2
- net /D5: track 0.00 -> 74.0 mm, vias 0 -> 3
- net Net-(D2-A): track 0.00 -> 70.2 mm, vias 0 -> 1
- net /D0: track 0.00 -> 66.8 mm, vias 0 -> 3
- net /RX: track 0.00 -> 62.4 mm, vias 0 -> 3
- net /A1: track 0.00 -> 62.0 mm, vias 0 -> 2
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