File: RE3RT4Prog.kicad_pcb (KiCad board)
At the start: 2 copper layers, 130 x 100 mm, 67 parts, among them J1 Conn_01x08, J2 Conn_01x08, J3 DE9_Receptacle_MountingHoles, J4 +5V, J5 GND, J6 PicKit, J7 Barrel_Jack_MountingPin, Q1 BD140, Q2 2N7000, Q3 2N7000, Q4 2N7000, U1 DG408, U2 155RE3, U3 556RT4, U4 74HC164, U6 PIC18F26K22-xSP, U7 MAX232, Y1 7.3728

Commit message: Work in progress
Parts:
- added R1: 1k, Resistor_THT:R_Axial_DIN0207_L6.3mm_D2.5mm_P10.16mm_Horizontal, F.Cu at (85.9, 75.6)
- added R4: 470, Resistor_THT:R_Axial_DIN0207_L6.3mm_D2.5mm_P10.16mm_Horizontal, F.Cu at (85.9, 79.7)
- R12, R21, R8: value R -> 1k
- R13: value R -> 100k
- R3, R7: value R -> 10k
- moved TP12 1.03 mm to (135.8, 58.0)
Connections:
- R3 pad 1: Net-(Q1-C) -> +12V
Other:
- outline, holes or cut-outs redrawn
